Commit message: hw 4

File: src/my_r2d2/urdf/r2d2.urdf.xacro (robot description, xacro)
@@ -228,4 +228,11 @@
     <origin rpy="0 1.57 0" xyz="0 0 0"/>
   </joint>
+  <link name="eye">
+  </link>
+  <joint name="eye_joint" type="fixed">
+    <parent link="lense"/>
+    <child link="eye"/>
+    <origin rpy="0 0 1.57"/>
+  </joint>
   <link name="base_footprint">
     <xacro:default_inertial mass="1000"/>
